File: drumTrigger4/drumtrigger4.sch (KiCad schematic (older format))
At the start: 23 parts, among them J1 Input, J2 TrigOut, J3 CVout, J4 Power, U1 TL074

Commit message: experimenting with adding input gain, likely swap input pot next
Parts:
- added J5: Gain, Connector_PinHeader_2.54mm:PinHeader_1x02_P2.54mm_Vertical, symbol Connector:Screw_Terminal_01x02
Connections:
- net at D2.2 (A), U1.1: now also J5.2 (Pin_2); no longer D1.2 (A), U1.2 (-)
- new net: D1.2 (A), J5.1 (Pin_1), U1.2 (-)
Changed lines of the file:
@@
 EESchema Schematic File Version 4
-EELAYER 30 0
+LIBS:drumtrigger4-cache
+EELAYER 26 0
 EELAYER END
 $Descr A4 11693 8268
@@
 $EndComp
 Wire Wire Line
-	3750 3200 3750 3500
+	3750 3200 3750 3400
 Wire Wire Line
 	3150 3500 3150 3300
@@
 Wire Wire Line
 	2950 3500 3150 3500
-Connection ~ 3150 3500
-Wire Wire Line
-	3150 3500 3750 3500
 $Comp
 L power:+12V #PWR0115
@@
 $EndComp
 Connection ~ 6050 3050
+$Comp
+L Connector:Screw_Terminal_01x02 J5
+U 1 1 5FC3FA6F
+P 3950 3500
+F 0 "J5" H 3868 3717 50  0000 C CNN
+F 1 "Gain" H 3868 3626 50  0000 C CNN
+F 2 "Connector_PinHeader_2.54mm:PinHeader_1x02_P2.54mm_Vertical" H 3950 3500 50  0001 C CNN
+F 3 "~" H 3950 3500 50  0001 C CNN
+	1    3950 3500
+	1    0    0    1
+$EndComp
+Wire Wire Line
+	3150 3500 3750 3500
+Connection ~ 3150 3500
 $EndSCHEMATC

Commit message: printed
Parts:
- removed RV1: InputTrim, Potentiometer_THT:Potentiometer_Piher_PT-6-V_Vertical, symbol Device:R_POT
- added R10, R11, R9: 10M, Resistor_THT:R_Axial_DIN0207_L6.3mm_D2.5mm_P10.16mm_Horizontal, symbol Device:R
- added R12: 1k, Resistor_THT:R_Axial_DIN0207_L6.3mm_D2.5mm_P10.16mm_Horizontal, symbol Device:R
- C1, C2: value 0.1uF -> 0.01uF
Connections:
- net GND: now also R11.2
- net at J1.1 (Pin_1): now also R12.2, R9.1
- net at U1.3 (+): now also R12.1
- new net: R10.1, R9.2
- new net: R10.2, R11.1
Other:
- moved on the sheet: C13, C14, J1, J4, U1E
